File: kicad/talon.kicad_pcb (KiCad board)
At the start: 2 copper layers, 82.9 x 110.6 mm, 23 parts, among them U1 nice_nano

Commit message: getting pretty tasty!
Parts:
- added REF**: through_hole_m2, footprints:through_hole_m2, F.Cu at (138.0, 75.5)
- added REF**: MountingHole_2.2mm_M2_DIN965_Pad, MountingHole:MountingHole_2.2mm_M2_DIN965_Pad, F.Cu at (119.0, 88.0)
- added REF**: MountingHole_2.2mm_M2_DIN965_Pad, MountingHole:MountingHole_2.2mm_M2_DIN965_Pad, F.Cu at (103.0, 125.5)
- added REF**: through_hole_m2, footprints:through_hole_m2, F.Cu at (157.0, 108.5)
- added REF**: MountingHole_2.2mm_M2_DIN965_Pad, MountingHole:MountingHole_2.2mm_M2_DIN965_Pad, F.Cu at (180.0, 125.5)
- added REF**: MountingHole_2.2mm_M2_DIN965_Pad, MountingHole:MountingHole_2.2mm_M2_DIN965_Pad, F.Cu at (161.0, 74.0)
- added REF**: Jumper_Open_0.8mm, footprints:Jumper_Open_0.8mm, F.Cu at (193.9, 44.4)
- added REF**: Jumper_Open_0.5mm, footprints:Jumper_Open_0.5mm, F.Cu at (186.2, 47.8)
- added REF**: MountingHole_2.2mm_M2_DIN965_Pad, MountingHole:MountingHole_2.2mm_M2_DIN965_Pad, F.Cu at (138.0, 113.5)
- added REF**: Jumper_Open_0.5mm, footprints:Jumper_Open_0.5mm, F.Cu at (192.9, 47.8)
- added REF**: through_hole_m2, footprints:through_hole_m2, F.Cu at (175.0, 74.0)
- added REF**: through_hole_m2, footprints:through_hole_m2, F.Cu at (122.5, 113.5)
- added REF**: MountingHole_2.2mm_M2_DIN965_Pad, MountingHole:MountingHole_2.2mm_M2_DIN965_Pad, F.Cu at (203.4, 141.5)
- added REF**: Jumper_Open_0.5mm, footprints:Jumper_Open_0.5mm, F.Cu at (189.6, 47.8)
- added REF**: through_hole_m2, footprints:through_hole_m2, F.Cu at (178.6, 142.0)
- REF** (x2): value Kailh_socket_MX_reversible -> locked
- moved REF** 2.21 mm to (108.8, 79.8)
- moved REF** 1.21 mm to (188.0, 77.0)
- moved U1 1.17 mm to (178.9, 57.9)
- renumbered REF** to locked
Other:
- board size 82.9 x 110.6 mm -> 84.1 x 110.6 mm
