File: kicad-slim/talon_slim.kicad_sch (KiCad schematic)
At the start: 36 parts, among them J1 JST connector, SW1 SW_Push, SW10 SW_Push, SW11 SW_Push, SW12 SW_Push, SW13 SW_Push, SW14 SW_Push, SW15 SW_Push, SW16 SW_Push, SW17 SW_Push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

Commit message: Slim looking not tooooo bad
Parts:
- added JP10, JP15, JP16, JP3: Jumper_2_Open, footprints:Jumper_Open_0.5mm, symbol Jumper:Jumper_2_Open
- added RESET_SW2: SW_Push, footprints:Panasonic_EVQPUL_EVQPUC, symbol Switch:SW_Push
- added SLIDE_SW2: SW_SPDT, footprints:SW_SSSS811101, symbol Switch:SW_SPDT
- J1: footprint footprints:power_connector -> Connector_JST:JST_PH_S2B-PH-K_1x02_P2.00mm_Horizontal
- RESET_SW1: footprint Button_Switch_THT:SW_PUSH_6mm -> footprints:Panasonic_EVQPUL_EVQPUC
- SLIDE_SW1: footprint footprints:slide_switch_5mm -> footprints:SW_SSSS811101
- SW1, SW10, SW11, SW12, SW13, SW14, SW15, SW16, SW17, SW2, SW3, SW4, SW5, SW6, SW7, SW9: footprint footprints:Kailh_socket_MX_reversible_1U -> footprints:SW_PG1350_reversible
- SW18, SW20: footprint footprints:Kailh_socket_MX_reversible_1_25U -> footprints:SW_PG1350_reversible_1.5U
- SW19, SW8: footprint footprints:Kailh_socket_MX_reversible_1_25U -> footprints:SW_PG1350_reversible
Connections:
- net BATIN: now also SLIDE_SW2.1 (A)
- net GND: now also JP15.2 (B), JP16.2 (B), RESET_SW2.2; no longer J1.2 (Pin_2)
- net RESET: now also RESET_SW2.1
- net at SLIDE_SW1.2 (B): now also JP10.2 (B); no longer J1.1 (Pin_1)
- new net: J1.2 (Pin_2), JP10.1 (A), JP15.1 (A)
- new net: JP3.2 (B), SLIDE_SW2.2 (B)
- new net: J1.1 (Pin_1), JP16.1 (A), JP3.1 (A)
Other:
- moved on the sheet: J1, RESET_SW1, SLIDE_SW1

Commit message: sent slim for procuction
Parts:
- SW20: footprint footprints:SW_PG1350_reversible_1.5U -> footprints:SW_PG1350_reversible
- SW8: footprint footprints:SW_PG1350_reversible -> footprints:SW_PG1350_reversible_1.5U
Changed lines of the file:
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@@
 			)
 		)
-		(property "Footprint" "footprints:SW_PG1350_reversible_1.5U"
+		(property "Footprint" "footprints:SW_PG1350_reversible"
 			(at 124.46 114.3 0)
 			(effects
@@
 			)
 		)
-		(property "Footprint" "footprints:SW_PG1350_reversible"
+		(property "Footprint" "footprints:SW_PG1350_reversible_1.5U"
 			(at 69.85 71.12 0)
 			(effects
